Commit message: Use .stl files instead of .STL

File: reflex_simulator/description/urdf/reflex/reflex.urdf.xacro (robot description, xacro)
@@ -77,5 +77,5 @@
         <origin xyz="-0.011 0.007 0.011" rpy="${pi} 0 0"/>
         <geometry>
-          <mesh filename="${mesh_path}/proximal.STL"/>
+          <mesh filename="${mesh_path}/proximal.stl"/>
         </geometry>
         <material name="black"/>
@@ -90,5 +90,5 @@
           <origin xyz="-0.011 0.007 0.011" rpy="${pi} 0 0"/>
           <geometry>
-            <mesh filename="${mesh_path}/proximal_coll.STL"/>
+            <mesh filename="${mesh_path}/proximal_coll.stl"/>
           </geometry>
         </collision>
@@ -105,5 +105,5 @@
         <origin xyz="${-0.077-flex_link_box_x/2} 0.007 ${0.007+flex_link_box_z/2+0.004+flex_z_offset}" rpy="${pi} 0 0"/>
         <geometry>
-          <mesh filename="${mesh_path}/distal.STL"/>
+          <mesh filename="${mesh_path}/distal.stl"/>
         </geometry>
         <material name="black"/>
@@ -118,5 +118,5 @@
           <origin xyz="${-0.077-flex_link_box_x/2} 0.007 ${0.007+flex_link_box_z/2}" rpy="${pi} 0 0"/>
           <geometry>
-            <mesh filename="${mesh_path}/distal_coll.STL"/>
+            <mesh filename="${mesh_path}/distal_coll.stl"/>
           </geometry>
         </collision>
@@ -132,5 +132,5 @@
         <origin xyz="-0.008 0.014 -0.002" rpy="${pi/2} ${pi/2} 0" />
         <geometry>
-          <mesh filename="${mesh_path}/proximal_pad.STL"/>
+          <mesh filename="${mesh_path}/proximal_pad.stl"/>
         </geometry>
         <material name="dark_grey"/>
@@ -145,5 +145,5 @@
           <origin xyz="-0.008 0.014 -0.002" rpy="${pi/2} ${pi/2} 0"/>
           <geometry>
-            <mesh filename="${mesh_path}/proximal_pad_coll.STL"/>
+            <mesh filename="${mesh_path}/proximal_pad_coll.stl"/>
           </geometry>
         </xacro:unless>
@@ -166,5 +166,5 @@
         <origin xyz="-0.008 0.0155 0.076" rpy="${pi/2} ${pi/2} 0"/>
         <geometry>
-          <mesh filename="${mesh_path}/distal_pad.STL"/>
+          <mesh filename="${mesh_path}/distal_pad.stl"/>
         </geometry>
         <material name="dark_grey"/>
@@ -179,5 +179,5 @@
           <origin xyz="-0.008 0.0155 0.076" rpy="${pi/2} ${pi/2} 0"/>
           <geometry>
-            <mesh filename="${mesh_path}/distal_pad_coll.STL"/>
+            <mesh filename="${mesh_path}/distal_pad_coll.stl"/>
           </geometry>
         </xacro:unless>
@@ -200,5 +200,5 @@
         <origin xyz="0 0 0" rpy="0 0 0"/>
         <geometry>
-          <mesh filename="${mesh_path}/swivel_${finger_id}.STL"/>
+          <mesh filename="${mesh_path}/swivel_${finger_id}.stl"/>
         </geometry>
         <material name="black"/>
@@ -213,5 +213,5 @@
           <origin xyz="0 0 0" rpy="0 0 0"/>
           <geometry>
-            <mesh filename="${mesh_path}/swivel_${finger_id}_coll.STL"/>
+            <mesh filename="${mesh_path}/swivel_${finger_id}_coll.stl"/>
           </geometry>
         </collision>
@@ -229,5 +229,5 @@
         <origin xyz="0 0 0" rpy="0 0 0"/>
         <geometry>
-          <mesh filename="${mesh_path}/base_link.STL"/>
+          <mesh filename="${mesh_path}/base_link.stl"/>
         </geometry>
         <material name="black"/>
@@ -242,5 +242,5 @@
           <origin xyz="0 0 0" rpy="0 0 0"/>
           <geometry>
-            <mesh filename="${mesh_path}/base_link_coll.STL"/>
+            <mesh filename="${mesh_path}/base_link_coll.stl"/>
           </geometry>
         </collision>
@@ -256,5 +256,5 @@
         <origin xyz="0 0 0" rpy="0 0 0"/>
         <geometry>
-          <mesh filename="${mesh_path}/pad.STL"/>
+          <mesh filename="${mesh_path}/pad.stl"/>
         </geometry>
         <material name="dark_grey"/>
@@ -269,5 +269,5 @@
           <origin xyz="0 0 0" rpy="0 0 0"/>
           <geometry>
-            <mesh filename="${mesh_path}/pad_coll.STL"/>
+            <mesh filename="${mesh_path}/pad_coll.stl"/>
           </geometry>
         </xacro:unless>

Commit message: Fix variable

File: reflex_simulator/description/urdf/reflex/reflex.urdf.xacro (robot description, xacro)
@@ -13,5 +13,5 @@
   </xacro:unless>
   <xacro:property name="pi" value="3.14159265359" />
-  <xacro:property name="mesh_path" value="package://description/meshes/reflex"/>
+  <xacro:property name="mesh_path" value="$(find description)/meshes/reflex"/>
   <xacro:include filename="$(find description)/urdf/xacro_macros/inertia_tensors.xacro"/>
   <!-- ===================================== MATERIALS ======================================= -->
