Commit message: Add modified intertia

File: reflex_simulator/description/urdf/environment/cylinder.urdf.xacro (robot description, xacro)
@@ -5,4 +5,6 @@
     <xacro:arg name="cylinder_radius" default="0.04"/>
     <xacro:arg name="cylinder_length" default="0.15"/>
+    <!-- inertia_scaling_factor = 1 means ground truth as calculated by formula -->
+    <xacro:arg name="inertia_scaling_factor" default="1"/>
     <xacro:property name="link_name" value="cylinder_link"/>
     <xacro:include filename="$(find description)/urdf/xacro_macros/inertia_tensors.xacro"/>
@@ -23,5 +25,5 @@
             <origin xyz="0 0 0" rpy="0 0 0"/>
             <mass value="$(arg cylinder_mass)"/>
-            <xacro:cylinder_inertia m="$(arg cylinder_mass)" r="$(arg cylinder_radius)" h="$(arg cylinder_length)"/>
+            <xacro:cylinder_inertia_mod m="$(arg cylinder_mass)" r="$(arg cylinder_radius)" h="$(arg cylinder_length)" scaling_factor="$(arg inertia_scaling_factor)"/>
         </inertial>
     </link>

File: reflex_simulator/description/urdf/xacro_macros/inertia_tensors.xacro (robot description, xacro)
@@ -23,3 +23,8 @@
 	     izz="${(1.0 / 2.0) * m * (r * r)}"/>
   </xacro:macro>
+  <xacro:macro name="cylinder_inertia_mod" params="m r h scaling_factor">
+    <inertia ixx="${(scaling_factor / 12.0) * m * (3 * r * r + h * h)}" ixy="0.0" ixz="0.0"
+	     iyy="${(scaling_factor / 12.0) * m * (3 * r * r + h * h)}" iyz="0.0"
+	     izz="${(scaling_factor / 2.0) * m * (r * r)}"/>
+  </xacro:macro>
 </robot>
