Commit message: Add scaling factor for cuboid inertia

File: reflex_simulator/description/urdf/environment/box.urdf.xacro (robot description, xacro)
@@ -6,4 +6,6 @@
     <xacro:arg name="box_y" default="0.08"/>
     <xacro:arg name="box_z" default="0.08"/>
+    <!-- inertia_scaling_factor = 1 means ground truth as calculated by formula -->
+    <xacro:arg name="inertia_scaling_factor" default="1"/>
     <xacro:property name="link_name" value="box_link"/>
     <xacro:include filename="$(find description)/urdf/xacro_macros/inertia_tensors.xacro"/>
@@ -24,5 +26,5 @@
             <origin xyz="0 0 0" rpy="0 0 0"/>
             <mass value="$(arg box_mass)"/>
-            <xacro:cuboid_inertia m="$(arg box_mass)" x="$(arg box_x)" y="$(arg box_y)" z="$(arg box_z)" />
+            <xacro:cuboid_inertia_mod m="$(arg box_mass)" x="$(arg box_x)" y="$(arg box_y)" z="$(arg box_z)" scaling_factor="$(arg inertia_scaling_factor)"/>
         </inertial>
     </link>

File: reflex_simulator/description/urdf/xacro_macros/inertia_tensors.xacro (robot description, xacro)
@@ -6,4 +6,9 @@
 	     iyy="${(1.0 / 12.0) * m * (x * x + z * z)}" iyz="0.0"
 	     izz="${(1.0 / 12.0) * m * (x * x + y * y)}"/>
+  </xacro:macro>
+  <xacro:macro name="cuboid_inertia_mod" params="m x y z scaling_factor">
+    <inertia ixx="${(scaling_factor / 12.0) * m * (y * y + z * z)}" ixy="0.0" ixz="0.0"
+	     iyy="${(scaling_factor / 12.0) * m * (x * x + z * z)}" iyz="0.0"
+	     izz="${(scaling_factor / 12.0) * m * (x * x + y * y)}"/>
   </xacro:macro>
   <xacro:macro name="ellipsoid_inertia" params="m x y z">
