Commit message: Introduce scaling factor for sphere inertia

File: reflex_simulator/description/urdf/environment/sphere.urdf.xacro (robot description, xacro)
@@ -4,4 +4,6 @@
     <xacro:arg name="sphere_mass" default="0.2"/>
     <xacro:arg name="sphere_radius" default="0.08"/>
+    <!-- inertia_scaling_factor = 1 means ground truth as calculated by formula -->
+    <xacro:arg name="inertia_scaling_factor" default="1"/>
     <xacro:property name="link_name" value="sphere_link"/>
     <xacro:include filename="$(find description)/urdf/xacro_macros/inertia_tensors.xacro"/>
@@ -22,5 +24,5 @@
             <origin xyz="0 0 0" rpy="0 0 0"/>
             <mass value="$(arg sphere_mass)"/>
-            <xacro:sphere_inertia m="$(arg sphere_mass)" r="$(arg sphere_radius)" />
+            <xacro:sphere_inertia_mod m="$(arg sphere_mass)" r="$(arg sphere_radius)" scaling_factor="$(arg inertia_scaling_factor)"/>
         </inertial>
     </link>

File: reflex_simulator/description/urdf/xacro_macros/inertia_tensors.xacro (robot description, xacro)
@@ -22,4 +22,9 @@
 	     izz="${(2.0 / 5.0) * m * (r * r)}"/>
   </xacro:macro>
+  <xacro:macro name="sphere_inertia_mod" params="m r scaling_factor">
+    <inertia ixx="${(scaling_factor * 2.0 / 5.0) * m * (r * r)}" ixy="0.0" ixz="0.0"
+	     iyy="${(scaling_factor * 2.0 / 5.0) * m * (r * r)}" iyz="0.0"
+	     izz="${(scaling_factor * 2.0 / 5.0) * m * (r * r)}"/>
+  </xacro:macro>
   <!-- Assuming z-axis goes along height of cylinder -->
   <xacro:macro name="cylinder_inertia" params="m r h">
